File: AnalogBoard.sch (EAGLE design)
At the start: 0 parts

Commit message: uploaded recent files.
Parts:
- added J1: 22-27-2021-02, con-molex:22-27-2021-02
- added J2: 22-27-2031-03, con-molex:22-27-2031-03
- added JP1: (no value), jumper:JP1E
- added LDR1, LDR2: (no value), SparkFun-Passives:RESISTORPTH-1/4W
- added LED1: (no value), led:LED3MM
- added PD1: BP104, opto-trans-siemens:BP104
Connections:
- new net 5V: J1-1.S, LDR1.2, PD1.A
- new net GND: J1-2.S, LDR2.1, LED1.C
- new net N$1: J2-2.S, JP1.1, LDR1.1
- new net N$2: LED1.A
- new net N$3: J2-3.S, JP1.2, LDR2.2
- new net N$5: J2-1.S, PD1.C
