File: DigitalBoard.sch (EAGLE design)
At the start: 0 parts

Commit message: uploaded recent files.
Parts:
- added D1, D2, D3, D4, D5, D6: (no value), SparkFun-LED:LED5MM
- added J3: 22-27-2021-02, con-molex:22-27-2021-02
- added JP1, JP2, JP3, JP4, JP5, JP6: (no value), jumper:JP1E
- added LED, SW: 22-27-2061-06, con-molex:22-27-2061-06
- added LOGO1: OSHW-LOGOS-COPPER, SparkFun-Aesthetics:OSHW-LOGOS-COPPER
- added SW1: (no value), special:SW_DIP-6
Connections:
- new net 5V: J3-1.S, SW1.1, SW1.2, SW1.3, SW1.4, SW1.5, SW1.6
- new net GND: D1.C, D2.C, D3.C, D4.C, D5.C, D6.C, J3-2.S
- new net N$1: JP1.1, SW-6.S, SW1.7
- new net N$10: JP4.2, LED-4.S
- new net N$11: JP5.2, LED-5.S
- new net N$12: JP6.2, LED-6.S
- new net N$13: D1.A
- new net N$14: D2.A
- new net N$15: D3.A
- new net N$16: D4.A
- new net N$17: D5.A
- new net N$18: D6.A
- new net N$2: JP2.1, SW-5.S, SW1.8
- new net N$3: JP3.1, SW-4.S, SW1.9
- new net N$4: JP4.1, SW-3.S, SW1.10
- new net N$5: JP5.1, SW-2.S, SW1.11
- new net N$6: JP6.1, SW-1.S, SW1.12
- new net N$7: JP1.2, LED-1.S
- new net N$8: JP2.2, LED-2.S
- new net N$9: JP3.2, LED-3.S
